File: AbeFrontPanel/AbePower.sch (KiCad schematic (older format))
At the start: 63 parts

Commit message: Rework again
Parts:
- U?: symbol AbeFrontPanel-rescue:MC33269D-3.3-MC33 -> MC33:MC33269D-3.3
- U?: symbol AbeFrontPanel-rescue:SN74ACT14D-SN74ACT14 -> SN74ACT14:SN74ACT14D
Changed lines of the file:
@@
 $EndDescr
 $Comp
-L AbeFrontPanel-rescue:MC33269D-3.3-MC33 U?
+L MC33:MC33269D-3.3 U?
 U 1 1 60812DCE
 P 2000 5000
@@
 $EndComp
 $Comp
-L AbeFrontPanel-rescue:SN74ACT14D-SN74ACT14 U?
+L SN74ACT14:SN74ACT14D U?
 U 1 1 6081383B
 P 6500 1100

Commit message: Rework Proj Structure
Parts:
- U?: symbol MC33:MC33269D-3.3 -> AbeFrontPanel-rescue:MC33269D-3.3-MC33
- U?: symbol SN74ACT14:SN74ACT14D -> AbeFrontPanel-rescue:SN74ACT14D-SN74ACT14
Changed lines of the file:
@@
 $EndDescr
 $Comp
-L MC33:MC33269D-3.3 U?
+L AbeFrontPanel-rescue:MC33269D-3.3-MC33 U?
 U 1 1 60812DCE
 P 2000 5000
@@
 $EndComp
 $Comp
-L SN74ACT14:SN74ACT14D U?
+L AbeFrontPanel-rescue:SN74ACT14D-SN74ACT14 U?
 U 1 1 6081383B
 P 6500 1100
