File: AbeFrontPanel/AbeMicrocontroller.sch (KiCad schematic (older format))
At the start: 15 parts

Commit message: Rework Proj Structure
Parts:
- U?: symbol MSP430:MSP430FR2475TRHAR -> AbeFrontPanel-rescue:MSP430FR2475TRHAR-MSP430
Changed lines of the file:
@@
 $EndDescr
 $Comp
-L MSP430:MSP430FR2475TRHAR U?
+L AbeFrontPanel-rescue:MSP430FR2475TRHAR-MSP430 U?
 U 1 1 6088B1A8
 P 5850 3850

Commit message: Rework again
Parts:
- U?: symbol AbeFrontPanel-rescue:MSP430FR2475TRHAR-MSP430 -> MSP430:MSP430FR2475TRHAR
Changed lines of the file:
@@
 $EndDescr
 $Comp
-L AbeFrontPanel-rescue:MSP430FR2475TRHAR-MSP430 U?
+L MSP430:MSP430FR2475TRHAR U?
 U 1 1 6088B1A8
 P 5850 3850
